Commit message: Updated description

File: urdf/four_wheels.xacro (robot description, xacro)
@@ -84,5 +84,5 @@
   </xacro:insertWheel>
   <xacro:property name="camera_size" value="0.02" />
-  <link name="camera_link">
+  <link name="front_camera">
     <collision>
       <origin xyz="0 0 0" rpy="0 0 0"/>
@@ -104,9 +104,9 @@
     </inertial>
   </link>
-  <joint name="camera_joint" type="fixed">
+  <joint name="front_camera_joint" type="fixed">
     <axis xyz="0 1 0"/>
     <origin xyz="0 ${base_length/2 + camera_size/2} ${base_height/2}" rpy="${PI} 0 ${PI/2}"/>
     <parent link="base_link"/>
-    <child link="camera_link"/>
+    <child link="front_camera"/>
   </joint>
   <link name="camera2_link">

File: urdf/rover.urdf (robot description, URDF)
Before this commit: robot rover, 16 links, 15 joints
Links:
- removed link camera_link
- added link arm_camera, mass 1e-5; collision box size=0.02 0.04 0.02; visual box size=0.02 0.04 0.02
- added link front_camera, mass 1e-5; collision box size=0.02 0.02 0.02; visual box size=0.02 0.04 0.04
Joints:
- removed joint camera_joint
- added joint arm_camera_joint: type fixed, parent fifth_link, child arm_camera, origin xyz=0 0 0.015 rpy=0 0 0, axis 0 1 0
- added joint front_camera_joint: type fixed, parent base_link, child front_camera, origin xyz=0 0.195 0.01975 rpy=3.1416 0 1.5708, axis 0 1 0
